File: pcb/airstream_controller.kicad_pcb (KiCad board)
At the start: 2 copper layers, 80 x 100 mm, 77 parts, among them J1 Prog, J2 Sensor 3 G C D, J3 Mot1, J4 Servo I 5 G, J5 Mot2, M1 Motor_DC, M2 Motor_DC, Q1 BC817, Q2 BC817, SW1 RESET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

Commit message: New Kicad Version
Routing:
- net Net-(R10-Pad2): track 28.1 -> 29.0 mm
